File: board/Pointcast_lower_board_V1.03.brd (EAGLE design)
At the start: 100.3 x 80 mm, 29 parts, among them U6 Ethernet, X2 3G module, X4 3GS shield

Commit message: V3.7.8 added temperature on main screen, dev and api switch on display, logging header with logs, retarts and fails
Parts:
- moved FRAME1 3.81 mm to (67.3, 66.7)
Routing:
- net PGM: track 0.00 -> 23.1 mm, vias 0 -> 3
- net D20: track 8.80 -> 9.53 mm
- net D17: track 13.8 -> 14.5 mm
- net D18: track 24.7 -> 25.4 mm
- net D19: track 19.7 -> 20.3 mm
- net D22: track 13.3 -> 13.9 mm
Changed lines of the file:
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@@
 <?xml version="1.0" encoding="utf-8"?>
 <!DOCTYPE eagle SYSTEM "eagle.dtd">
-<eagle version="7.4.0">
+<eagle version="7.5.0">
 <drawing>
 <settings>
@@
 <hole x="2.54" y="2.54" drill="3.2"/>
 <hole x="2.54" y="77.47" drill="3.2"/>
-<text x="53.975" y="71.755" size="1.27" layer="51">POINTCAST V2.0</text>
-<text x="46.365628125" y="1.366353125" size="1.016" layer="51">Thanks to Shuttleworth Foundation, Medcom and Safecast volunteers</text>
+<text x="53.975" y="71.755" size="1.016" layer="51">POINTCAST V2.0</text>
+<text x="46.365628125" y="1.366353125" size="0.762" layer="51">Thanks to Shuttleworth Foundation, Medcom and Safecast volunteers</text>
 </plain>
 <attributes>
 <attribute name="DESIGNER" value="Rob Oudendijk"/>
-<attribute name="VERSION" value="Rev 1.02"/>
+<attribute name="VERSION" value="Rev 1.03"/>
 </attributes>
 <variantdefs>
@@
 <attribute name="NAME" x="47.18228125" y="5.983909375" size="1.27" layer="21" rot="R90"/>
 </element>
-<element name="FRAME1" library="SparkFun-Aesthetics" package="CREATIVE_COMMONS" value="FRAME-LEDGER" x="71.12" y="66.675" smashed="yes">
+<element name="FRAME1" library="SparkFun-Aesthetics" package="CREATIVE_COMMONS" value="FRAME-LEDGER" x="67.31" y="66.675" smashed="yes">
 <attribute name="VERSION" x="82.55" y="71.755" size="1.27" layer="51" font="vector"/>
 </element>
@@
 <via x="20.6248" y="75.565" extent="1-16" drill="0.6096"/>
 <contactref element="TEENSY" pad="23/A9"/>
-<wire x1="11.43" y1="71.12" x2="11.557" y2="71.12" width="0" layer="19" extent="16-16"/>
+<wire x1="11.557" y1="71.12" x2="11.43" y2="71.12" width="0.4064" layer="16"/>
 </signal>
 <signal name="D22">
@@
 <via x="19.558" y="72.898" extent="1-16" drill="0.6096"/>
 <contactref element="TEENSY" pad="22/A8"/>
-<wire x1="13.97" y1="71.12" x2="14.5796" y2="71.12" width="0" layer="19" extent="1-1"/>
+<wire x1="14.5796" y1="71.12" x2="13.97" y2="71.12" width="0.4064" layer="1"/>
 </signal>
 <signal name="D21">
@@
 <wire x1="20.2692" y1="77.343" x2="20.32" y2="77.47" width="0.4064" layer="1"/>
 <contactref element="TEENSY" pad="21/A7"/>
-<wire x1="16.51" y1="71.12" x2="16.5354" y2="71.12" width="0" layer="19" extent="1-1"/>
+<wire x1="16.5354" y1="71.12" x2="16.51" y2="71.12" width="0.4064" layer="1"/>
 </signal>
 <signal name="D20">
@@
 <via x="15.4686" y="73.4314" extent="1-16" drill="0.6096"/>
 <contactref element="TEENSY" pad="20/A6"/>
-<wire x1="18.3134" y1="71.12" x2="19.05" y2="71.12" width="0" layer="19" extent="16-16"/>
+<wire x1="18.3134" y1="71.12" x2="19.05" y2="71.12" width="0.4064" layer="16"/>
 </signal>
 <signal name="D17">
@@
 <via x="18.3134" y="74.8538" extent="1-16" drill="0.6096"/>
 <contactref element="TEENSY" pad="17/A3"/>
-<wire x1="26.67" y1="71.8312" x2="26.67" y2="71.12" width="0" layer="19" extent="16-16"/>
+<wire x1="26.67" y1="71.8312" x2="26.67" y2="71.12" width="0.4064" layer="16"/>
 </signal>
 <signal name="D18">
@@
 <wire x1="10.1346" y1="77.343" x2="10.16" y2="77.47" width="0.4064" layer="1"/>
 <contactref element="TEENSY" pad="18/A4"/>
-<wire x1="23.4696" y1="71.12" x2="24.13" y2="71.12" width="0" layer="19" extent="1-1"/>
+<wire x1="23.4696" y1="71.12" x2="24.13" y2="71.12" width="0.4064" layer="1"/>
 </signal>
 <signal name="D19">
@@
 <wire x1="12.8016" y1="77.343" x2="12.7" y2="77.47" width="0.4064" layer="16"/>
 <contactref element="TEENSY" pad="19/A5"/>
-<wire x1="20.9804" y1="71.12" x2="21.59" y2="71.12" width="0" layer="19" extent="16-16"/>
+<wire x1="20.9804" y1="71.12" x2="21.59" y2="71.12" width="0.4064" layer="16"/>
 </signal>
 <signal name="D13">
@@
 <contactref element="JP3" pad="16"/>
 <contactref element="TEENSY" pad="PGM"/>
-<wire x1="36.83" y1="66.04" x2="48.26" y2="77.47" width="0" layer="19" extent="1-1"/>
+<wire x1="39.8272" y1="66.1416" x2="36.9824" y2="66.1416" width="0.4064" layer="1"/>
+<wire x1="41.2496" y1="67.564" x2="39.8272" y2="66.1416" width="0.4064" layer="1"/>
+<wire x1="42.1386" y1="67.564" x2="41.2496" y2="67.564" width="0.4064" layer="16"/>
+<wire x1="43.561" y1="66.1416" x2="42.1386" y2="67.564" width="0.4064" layer="16"/>
+<wire x1="45.6946" y1="68.2752" x2="43.561" y2="66.1416" width="0.4064" layer="1"/>
+<wire x1="43.3832" y1="70.5866" x2="45.6946" y2="68.2752" width="0.4064" layer="16"/>
+<wire x1="43.3832" y1="72.5424" x2="43.3832" y2="70.5866" width="0.4064" layer="16"/>
+<wire x1="48.1838" y1="77.343" x2="43.3832" y2="72.5424" width="0.4064" layer="16"/>
+<wire x1="36.9824" y1="66.1416" x2="36.83" y2="66.04" width="0.4064" layer="1"/>
+<wire x1="48.1838" y1="77.343" x2="48.26" y2="77.47" width="0.4064" layer="16"/>
+<via x="41.2496" y="67.564" extent="1-16" drill="0.6096"/>
+<via x="43.561" y="66.1416" extent="1-16" drill="0.6096"/>
+<via x="45.6946" y="68.2752" extent="1-16" drill="0.6096"/>
 </signal>
 </signals>
